Commit message: nb

File: src/my_nav2_robot/urdf/robot.urdf.xacro (robot description, xacro)
@@ -118,4 +118,14 @@
             <material name="red"/>
         </visual>
+        <!--
+        <collision>
+            <geometry>
+                <cylinder radius="${laser_radius}" length="${laser_height}"/>
+            </geometry>
+        </collision>
+        -->
+        <xacro:inertial_cylinder mass="0.1" r="${laser_radius}" h="${laser_height}">
+            <origin xyz="0 0 0" rpy="0 0 0"/>
+        </xacro:inertial_cylinder>
     </link>
     <joint name="laser_joint" type="fixed">
@@ -124,3 +134,51 @@
         <origin xyz="0 0 ${chassis_height + laser_height / 2}" rpy="0 0 0"/>
     </joint>
+    <gazebo reference="laser_link">
+        <sensor name="gpu_lidar" type="gpu_lidar">
+            <topic>scan</topic>
+            <pose>0 0 0 0 0 0</pose>
+            <frame_id>laser_link</frame_id>
+            <gz_frame_id>laser_link</gz_frame_id>
+            <visualize>true</visualize> <update_rate>10</update_rate>
+            <lidar>
+                <scan>
+                    <horizontal>
+                        <samples>360</samples>
+                        <resolution>1</resolution>
+                        <min_angle>-3.14159</min_angle>
+                        <max_angle>3.14159</max_angle>
+                    </horizontal>
+                </scan>
+                <range>
+                    <min>0.12</min>
+                    <max>12.0</max>
+                    <resolution>0.01</resolution>
+                </range>
+            </lidar>
+            <plugin filename="gz-sim-sensors-system" name="gz::sim::systems::Sensors">
+                <render_engine>ogre2</render_engine>
+            </plugin>
+        </sensor>
+    </gazebo>
+    <gazebo>
+        <plugin
+            filename="gz-sim-diff-drive-system"
+            name="gz::sim::systems::DiffDrive">
+            <left_joint>front_left_wheel_joint</left_joint>
+            <right_joint>front_right_wheel_joint</right_joint>
+            <wheel_separation>${chassis_width + wheel_width}</wheel_separation>
+            <wheel_radius>${wheel_radius}</wheel_radius>
+            <topic>cmd_vel</topic>
+            <odom_topic>odom</odom_topic>
+            <frame_id>odom</frame_id>
+            <child_frame_id>base_footprint</child_frame_id>
+            <publish_odom_tf>true</publish_odom_tf>
+            <use_gz_time>true</use_gz_time>
+        </plugin>
+        <plugin
+            filename="gz-sim-joint-state-publisher-system"
+            name="gz::sim::systems::JointStatePublisher">
+            <topic>joint_states</topic>
+        </plugin>
+    </gazebo>
 </robot>

Commit message: 视觉里程计1

File: src/my_nav2_robot/urdf/robot.urdf.xacro (robot description, xacro)
@@ -15,4 +15,7 @@
     <xacro:property name="laser_radius" value="0.03"/>
     <xacro:property name="laser_height" value="0.04"/>
+    <!--深度相机形态-->
+    <xacro:property name="camera_radius" value="0.03"/>
+    <xacro:property name="camera_height" value="0.04"/>
     <!--机器人机身的物理属性-->
     <xacro:macro name="inertial_box" params="mass l w h *origin">
@@ -118,11 +121,4 @@
             <material name="red"/>
         </visual>
-        <!--
-        <collision>
-            <geometry>
-                <cylinder radius="${laser_radius}" length="${laser_height}"/>
-            </geometry>
-        </collision>
-        -->
         <xacro:inertial_cylinder mass="0.1" r="${laser_radius}" h="${laser_height}">
             <origin xyz="0 0 0" rpy="0 0 0"/>
@@ -134,4 +130,23 @@
         <origin xyz="0 0 ${chassis_height + laser_height / 2}" rpy="0 0 0"/>
     </joint>
+    <!--深度相机-->
+    <!--物理位置-->
+    <link name="camera_link">
+        <visual>
+            <geometry>
+                <cylinder radius="${laser_radius}" length="${laser_height}"/>
+            </geometry>
+            <material name="blue"/>
+        </visual>
+        <xacro:inertial_cylinder mass="0.1" r="${laser_radius}" h="${laser_height}">
+            <origin xyz="0 0 0" rpy="0 0 0"/>
+        </xacro:inertial_cylinder>
+    </link>
+    <joint name="camera_joint" type="fixed">
+        <parent link="base_link"/>
+        <child link="camera_link"/>
+        <origin xyz="0.2 0 ${chassis_height + laser_height / 2 - 0.06}" rpy="0 0 0"/>
+    </joint>
+    <!--雷达插件-->
     <gazebo reference="laser_link">
         <sensor name="gpu_lidar" type="gpu_lidar">
@@ -156,16 +171,15 @@
                 </range>
             </lidar>
-            <plugin filename="gz-sim-sensors-system" name="gz::sim::systems::Sensors">
-                <render_engine>ogre2</render_engine>
-            </plugin>
         </sensor>
-        <sensor name="camera" type="camera">
-            <pose>0.2 0 0.2 0 0 0</pose> <update_rate>30</update_rate>
-            <frame_id>laser_link</frame_id>
-            <gz_frame_id>laser_link</gz_frame_id>
+    </gazebo>
+    <!--深度相机插件-->
+    <gazebo reference="camera_link">
+        <sensor name="depth_camera" type="rgbd_camera">
             <visualize>true</visualize>
-            <topic>camera/image_raw</topic>
+            <update_rate>10.0</update_rate>
+            <topic>depth_camera</topic>
+            <gz_frame_id>camera_link</gz_frame_id>
             <camera>
-                <horizontal_fov>1.089</horizontal_fov>
+                <horizontal_fov>1.047198</horizontal_fov>
                 <image>
                     <width>640</width>
@@ -174,9 +188,15 @@
                 </image>
                 <clip>
-                    <near>0.05</near>
-                    <far>8.0</far>
+                    <near>0.1</near>
+                    <far>5.0</far>
                 </clip>
             </camera>
         </sensor>
+    </gazebo>
+    <!--全局挂载插件-->
+    <gazebo>
+        <plugin filename="gz-sim-sensors-system" name="gz::sim::systems::Sensors">
+            <render_engine>ogre2</render_engine>
+        </plugin>
     </gazebo>
     <gazebo reference="front_left_wheel_link">

Commit message: osqp+漂移问题修正

File: src/my_nav2_robot/urdf/robot.urdf.xacro (robot description, xacro)
@@ -148,4 +148,21 @@
         <origin xyz="0.2 0 ${chassis_height + laser_height / 2 - 0.06}" rpy="0 0 0"/>
     </joint>
+    <!--imu-->
+    <link name = "imu_link">
+        <visual>
+            <geometry>
+                <box size = "0.02 0.02 0.02"/>
+            </geometry>
+            <material name = "black"/>
+        </visual>
+        <xacro:inertial_box mass="0.01" l="0.02" w="0.02" h="0.02">
+            <origin xyz="0 0 0" rpy="0 0 0"/>
+        </xacro:inertial_box>
+    </link>
+    <joint name = "imu_joint" type = "fixed">
+        <parent link = "base_link"/>
+        <child link = "imu_link"/>
+        <origin xyz="0 0 0" rpy="0 0 0"/>
+    </joint>
     <!--雷达插件-->
     <gazebo reference="laser_link">
@@ -177,5 +194,5 @@
         <sensor name="depth_camera" type="rgbd_camera">
             <visualize>true</visualize>
-            <update_rate>10.0</update_rate>
+            <update_rate>1.0</update_rate> <!-- 原10hz，到时候再改回来 -->
             <topic>depth_camera</topic>
             <gz_frame_id>camera_link</gz_frame_id>
@@ -194,4 +211,12 @@
         </sensor>
     </gazebo>
+    <!--imu插件-->
+    <gazebo reference="imu_link">
+        <sensor name="imu" type="imu">
+            <update_rate>1.0</update_rate> <!-- 原100hz，到时候再改回来 -->
+            <topic>imu</topic>
+            <gz_frame_id>imu_link</gz_frame_id>
+        </sensor>
+    </gazebo>
     <!--全局挂载插件-->
     <gazebo>
@@ -199,4 +224,5 @@
             <render_engine>ogre2</render_engine>
         </plugin>
+        <plugin filename="gz-sim-imu-system" name="gz::sim::systems::Imu"/>
     </gazebo>
     <gazebo reference="front_left_wheel_link">
@@ -224,5 +250,5 @@
             <left_joint>rear_left_wheel_joint</left_joint>
             <right_joint>rear_right_wheel_joint</right_joint>
-            <wheel_separation>0.52</wheel_separation>
+            <wheel_separation>0.34</wheel_separation>
             <wheel_radius>${wheel_radius}</wheel_radius>
             <max_wheel_torque>50</max_wheel_torque>
@@ -230,12 +256,7 @@
             <topic>cmd_vel</topic>
             <odom_topic>odom</odom_topic>
-            <tf_topic>/tf</tf_topic> <!--重要-->
+            <tf_topic>/wheel_tf</tf_topic> <!--可以不开，专门给轮式里程计的，不写tf是为了防止跟轮式里程计抢发布-->
             <frame_id>odom</frame_id>
             <child_frame_id>base_footprint</child_frame_id>
-            <publish_odom>true</publish_odom>
-            <publish_odom_tf>false</publish_odom_tf>
-            <publish_wheel_tf>true</publish_wheel_tf>
-            <odometry_frame>odom</odometry_frame>
-            <use_gz_time>true</use_gz_time>
         </plugin>
         <plugin
@@ -249,7 +270,8 @@
             filename="gz-sim-odometry-publisher-system"
             name="gz::sim::systems::OdometryPublisher">
-            <odom_topic>ground_truth</odom_topic> <odom_frame>world</odom_frame>
+            <odom_topic>ground_truth</odom_topic>  <!--里程计请用此话题！！！-->
+            <odom_frame>odom</odom_frame>
             <robot_base_frame>base_footprint</robot_base_frame>
-            <tf_topic>ground_truth/tf</tf_topic>
+            <tf_topic>/tf</tf_topic>
             <dimensions>3</dimensions>
         </plugin>

Commit message: 麦克纳姆轮

File: src/my_nav2_robot/urdf/robot.urdf.xacro (robot description, xacro)
@@ -7,5 +7,5 @@
     <!--轮子形态-->
     <xacro:property name="wheel_radius" value="0.05"/>
-    <xacro:property name="wheel_width" value="0.04"/>
+    <xacro:property name="wheel_width" value="0.025"/>
     <!--轮子位置-->
     <xacro:property name="wheel_offset_x" value="${chassis_length / 2 - 0.05}"/>
@@ -83,20 +83,20 @@
         <link name="${prefix}_wheel_link">
             <visual>
-                <!--roll需要为pi/2的原因是圆柱体默认朝z轴向上-->
-                <origin xyz="0 0 0" rpy="${pi/2} 0 0"/>
+                <!--roll需要为pi/2的原因是圆柱体默认朝z轴向上，额这是之前的圆柱体代码，换成麦轮就不一样了-->
+                <origin xyz="0 0 -0.05" rpy="0 0 0"/>
                 <geometry>
                     <!--圆柱体-->
-                    <cylinder radius="${wheel_radius}" length="${wheel_width}"/>
+                    <mesh filename="package://my_nav2_robot/meshes/mecanum_${prefix}_hands.stl" scale="0.001 0.001 0.001"/>
                 </geometry>
                 <material name="black"/>
             </visual>
             <collision>
-                <origin xyz="0 0 0" rpy="${pi/2} 0 0"/>
+                <origin xyz="0 0 -0.05" rpy="0 0 0"/>
                 <geometry>
-                    <cylinder radius="${wheel_radius}" length="${wheel_width}"/>
+                    <mesh filename="package://my_nav2_robot/meshes/mecanum_${prefix}_hands.stl" scale="0.001 0.001 0.001"/>
                 </geometry>
             </collision>
             <xacro:inertial_cylinder mass="0.5" r="${wheel_radius}" h="${wheel_width}">
-                <origin xyz="0 0 0" rpy="${pi/2} 0 0"/>
+                <origin xyz="0 0 -0.05" rpy="0 0 0"/>
             </xacro:inertial_cylinder>
         </link>
@@ -107,5 +107,16 @@
             <!--旋转轴-->
             <axis xyz="0 1 0"/>
+            <limit effort="50" velocity="50"/>
+            <dynamics damping="0.0" friction="0.05"/>
         </joint>
+        <gazebo reference="${prefix}_wheel_link">
+            <mu1>2.0</mu1>
+            <mu2>0.5</mu2>
+            <kp>1000000.0</kp>
+            <kd>1.0</kd>
+            <fdir1>1 0 0</fdir1>
+            <minDepth>0.001</minDepth>
+            <material>Gazebo/Black</material>
+        </gazebo>
     </xacro:macro>
     <xacro:wheel prefix="front_left" reflect_x="1" reflect_y="1"/>
@@ -226,21 +237,6 @@
         <plugin filename="gz-sim-imu-system" name="gz::sim::systems::Imu"/>
     </gazebo>
-    <gazebo reference="front_left_wheel_link">
-        <mu1>1.5</mu1>
-        <mu2>1.5</mu2>
-    </gazebo>
-    <gazebo reference="front_right_wheel_link">
-        <mu1>1.5</mu1>
-        <mu2>1.5</mu2>
-    </gazebo>
-    <gazebo reference="rear_left_wheel_link">
-        <mu1>1.5</mu1>
-        <mu2>1.5</mu2>
-    </gazebo>
-    <gazebo reference="rear_right_wheel_link">
-        <mu1>1.5</mu1>
-        <mu2>1.5</mu2>
-    </gazebo>
-    <gazebo>
+    <!-- 差速驱动插件 -->
+    <!-- <gazebo>
         <plugin
             filename="gz-sim-diff-drive-system"
@@ -256,5 +252,5 @@
             <topic>cmd_vel</topic>
             <odom_topic>odom</odom_topic>
-            <tf_topic>/wheel_tf</tf_topic> <!--可以不开，专门给轮式里程计的，不写tf是为了防止跟轮式里程计抢发布-->
+            <tf_topic>/wheel_tf</tf_topic>
             <frame_id>odom</frame_id>
             <child_frame_id>base_footprint</child_frame_id>
@@ -265,4 +261,41 @@
             <topic>joint_states</topic>
         </plugin>
+    </gazebo> -->
+    <!-- 麦克纳姆轮（何用？） -->
+    <!-- <gazebo>
+        <plugin
+            filename = "gz-sim-mecanum-drive-system"
+            name = "gz::sim::systems::MecanumDrive">
+            <front_left_joint>front_left_wheel_joint</front_left_joint>
+            <front_right_joint>front_right_wheel_joint</front_right_joint>
+            <back_left_joint>rear_left_wheel_joint</back_left_joint>
+            <back_right_joint>rear_right_wheel_joint</back_right_joint>
+            <wheel_separation>${chassis_width + wheel_width}</wheel_separation>
+            <wheel_radius>${wheel_radius}</wheel_radius>
+            <wheel_base>${2 * wheel_offset_y}</wheel_base>
+            <topic>/cmd_vel</topic>
+            <odom_topic>/odom</odom_topic>
+            <tf_topic>/wheel_tf</tf_topic>
+            <frame_id>odom</frame_id>
+            <child_frame_id>base_footprint</child_frame_id>
+        </plugin>
+        <plugin
+            filename="gz-sim-joint-state-publisher-system"
+            name="gz::sim::systems::JointStatePublisher">
+            <topic>/joint_states</topic>
+        </plugin>
+    </gazebo> -->
+    <!-- 代替麦克纳姆轮的直接移动插件 -->
+    <gazebo>
+        <plugin
+            filename = "gz-sim-velocity-control-system"
+            name = "gz::sim::systems::VelocityControl">
+            <topic>/cmd_vel</topic>
+        </plugin>
+        <plugin
+            filename="gz-sim-joint-state-publisher-system"
+            name="gz::sim::systems::JointStatePublisher">
+            <topic>/joint_states</topic>
+        </plugin>
     </gazebo>
     <gazebo>
@@ -270,5 +303,5 @@
             filename="gz-sim-odometry-publisher-system"
             name="gz::sim::systems::OdometryPublisher">
-            <odom_topic>ground_truth</odom_topic>  <!--里程计请用此话题！！！-->
+            <odom_topic>/ground_truth</odom_topic>  <!--里程计请用此话题！！！-->
             <odom_frame>odom</odom_frame>
             <robot_base_frame>base_footprint</robot_base_frame>

Commit message: some big change

File: src/my_nav2_robot/urdf/robot.urdf.xacro (robot description, xacro)
@@ -84,19 +84,24 @@
             <visual>
                 <!--roll需要为pi/2的原因是圆柱体默认朝z轴向上，额这是之前的圆柱体代码，换成麦轮就不一样了-->
-                <origin xyz="0 0 -0.05" rpy="0 0 0"/>
+                <!-- <origin xyz="0 0 -0.05" rpy="0 0 0"/>
+                <geometry>
+                    <mesh filename="package://my_nav2_robot/meshes/mecanum_${prefix}_hands.stl" scale="0.001 0.001 0.001"/>
+                </geometry> -->
+                <origin xyz="0 0 0" rpy="${pi / 2} 0 0"/>
                 <geometry>
                     <!--圆柱体-->
-                    <mesh filename="package://my_nav2_robot/meshes/mecanum_${prefix}_hands.stl" scale="0.001 0.001 0.001"/>
+                    <cylinder radius="${wheel_radius}" length="${wheel_width}"/>
                 </geometry>
                 <material name="black"/>
             </visual>
             <collision>
-                <origin xyz="0 0 -0.05" rpy="0 0 0"/>
+                <origin xyz="0 0 0" rpy="${pi / 2} 0 0"/>
                 <geometry>
-                    <mesh filename="package://my_nav2_robot/meshes/mecanum_${prefix}_hands.stl" scale="0.001 0.001 0.001"/>
+                    <!--圆柱体-->
+                    <cylinder radius="${wheel_radius}" length="${wheel_width}"/>
                 </geometry>
             </collision>
             <xacro:inertial_cylinder mass="0.5" r="${wheel_radius}" h="${wheel_width}">
-                <origin xyz="0 0 -0.05" rpy="0 0 0"/>
+                <origin xyz="0 0 0" rpy="${pi / 2} 0 0"/>
             </xacro:inertial_cylinder>
         </link>
@@ -108,5 +113,5 @@
             <axis xyz="0 1 0"/>
             <limit effort="50" velocity="50"/>
-            <dynamics damping="0.0" friction="0.05"/>
+            <dynamics damping="0.1" friction="0.1"/>
         </joint>
         <gazebo reference="${prefix}_wheel_link">
@@ -115,7 +120,4 @@
             <kp>1000000.0</kp>
             <kd>1.0</kd>
-            <fdir1>1 0 0</fdir1>
-            <minDepth>0.001</minDepth>
-            <material>Gazebo/Black</material>
         </gazebo>
     </xacro:macro>
@@ -205,5 +207,5 @@
         <sensor name="depth_camera" type="rgbd_camera">
             <visualize>true</visualize>
-            <update_rate>1.0</update_rate> <!-- 原10hz，到时候再改回来 -->
+            <update_rate>10.0</update_rate> <!-- 原10hz，到时候再改回来 -->
             <topic>depth_camera</topic>
             <gz_frame_id>camera_link</gz_frame_id>
@@ -225,5 +227,5 @@
     <gazebo reference="imu_link">
         <sensor name="imu" type="imu">
-            <update_rate>1.0</update_rate> <!-- 原100hz，到时候再改回来 -->
+            <update_rate>100.0</update_rate> <!-- 原100hz，到时候再改回来 -->
             <topic>imu</topic>
             <gz_frame_id>imu_link</gz_frame_id>
